Commit message: diet

File: craft/go2_colored.urdf (robot description, URDF)
Before this commit: robot go2_arm, 46 links, 45 joints
Links:
- removed link camera
- removed link gripper_base
- removed link gripper_claw_left
- removed link gripper_claw_right
- removed link housing
- removed link node0
- removed link node1
- removed link node2
- removed link node3
- removed link node4
- removed link node5
- removed link node6
- removed link node7
- removed link node8
- removed link node9
- removed link plate
- removed link wedge
Joints:
- removed joint j_go2_base_arm_plate
- removed joint j_gripper_base_camera
- removed joint j_gripper_base_claw_left
- removed joint j_gripper_base_claw_right
- removed joint j_housing_wedge
- removed joint j_node0_node1
- removed joint j_node1_node2
- removed joint j_node2_node3
- removed joint j_node3_node4
- removed joint j_node4_node5
- removed joint j_node5_node6
- removed joint j_node6_node7
- removed joint j_node7_node8
- removed joint j_node8_node9
- removed joint j_node9_gripper_base
- removed joint j_plate_housing
- removed joint j_wedge_node0
