Commit message: merged

File: craft/robot.urdf (robot description, URDF)
Before this commit: robot Robot, 16 links, 15 joints
Joints:
- joint j_node9_gripper_base: origin xyz=0.05 0 0 rpy=0 -1.57079633 0 -> xyz=0.05 -0.012 0 rpy=0 -1.57079633 0

Commit message: troit

File: craft/robot.urdf (robot description, URDF)
Before this commit: robot Robot, 16 links, 15 joints
Links:
- link gripper_base: mass 0.2 -> 0.15
- link gripper_claw_left: mass 0.3 -> 0.05
- link gripper_claw_right: mass 0.3 -> 0.05
- link housing: mass 3 -> 0.5
- link node0: mass 0.1 -> 0.05
- link node1: mass 0.1 -> 0.05
- link node2: mass 0.1 -> 0.05
- link node3: mass 0.1 -> 0.05
- link node4: mass 0.1 -> 0.05
- link node5: mass 0.1 -> 0.05
- link node6: mass 0.1 -> 0.05
- link node7: mass 0.1 -> 0.05
- link node8: mass 0.1 -> 0.05
- link node9: mass 0.1 -> 0.05
- link plate: mass 10 -> 0.5

Commit message: update

File: craft/robot.urdf (robot description, URDF)
Before this commit: robot Robot, 16 links, 15 joints
Links:
- link housing: mass 0.5 -> 1.8
- link node0: mass 0.05 -> 0.15
- link node1: mass 0.05 -> 0.15
- link node2: mass 0.05 -> 0.15
- link node3: mass 0.05 -> 0.15
- link node4: mass 0.05 -> 0.15
- link node5: mass 0.05 -> 0.15
- link node6: mass 0.05 -> 0.15
- link node7: mass 0.05 -> 0.15
- link node8: mass 0.05 -> 0.15
- link node9: mass 0.05 -> 0.15
- link plate: mass 0.5 -> 1.5

Commit message: update

File: craft/robot.urdf (robot description, URDF)
Before this commit: robot Robot, 16 links, 15 joints
Links:
- added link FL_calf, mass 0.154; collision cylinder length=0.12 radius=0.012; visual mesh filename=dae/calf.dae
- added link FL_calflower; collision cylinder length=0.065 radius=0.011
- added link FL_calflower1; collision cylinder length=0.03 radius=0.0155
- added link FL_foot, mass 0.04; collision sphere radius=0.022; visual mesh filename=dae/foot.dae
- added link FL_hip, mass 0.678; collision cylinder length=0.04 radius=0.046; visual mesh filename=dae/hip.dae
- added link FL_thigh, mass 1.152; collision box size=0.11 0.0245 0.034; visual mesh filename=dae/thigh.dae
- added link FR_calf, mass 0.154; collision cylinder length=0.12 radius=0.013; visual mesh filename=dae/calf_mirror.dae
- added link FR_calflower; collision cylinder length=0.065 radius=0.011
- added link FR_calflower1; collision cylinder length=0.03 radius=0.0155
- added link FR_foot, mass 0.04; collision sphere radius=0.022; visual mesh filename=dae/foot.dae
- added link FR_hip, mass 0.678; collision cylinder length=0.04 radius=0.046; visual mesh filename=dae/hip.dae
- added link FR_thigh, mass 1.152; collision box size=0.11 0.0245 0.034; visual mesh filename=dae/thigh_mirror.dae
- added link Head_lower, mass 0.001; collision sphere radius=0.047
- added link Head_upper, mass 0.001; collision cylinder length=0.09 radius=0.05
- added link RL_calf, mass 0.154; collision cylinder length=0.12 radius=0.013; visual mesh filename=dae/calf.dae
- added link RL_calflower; collision cylinder length=0.065 radius=0.011
- added link RL_calflower1; collision cylinder length=0.03 radius=0.0155
- added link RL_foot, mass 0.04; collision sphere radius=0.022; visual mesh filename=dae/foot.dae
- added link RL_hip, mass 0.678; collision cylinder length=0.04 radius=0.046; visual mesh filename=dae/hip.dae
- added link RL_thigh, mass 1.152; collision box size=0.11 0.0245 0.034; visual mesh filename=dae/thigh.dae
- added link RR_calf, mass 0.154; collision cylinder length=0.12 radius=0.013; visual mesh filename=dae/calf_mirror.dae
- added link RR_calflower; collision cylinder length=0.065 radius=0.011
- added link RR_calflower1; collision cylinder length=0.03 radius=0.0155
- added link RR_foot, mass 0.04; collision sphere radius=0.022; visual mesh filename=dae/foot.dae
- added link RR_hip, mass 0.678; collision cylinder length=0.04 radius=0.046; visual mesh filename=dae/hip.dae
- added link RR_thigh, mass 1.152; collision box size=0.11 0.0245 0.034; visual mesh filename=dae/thigh_mirror.dae
- added link base, mass 6.921; collision box size=0.3762 0.0935 0.114; visual mesh filename=dae/base.dae
- added link imu, mass 0
- added link radar, mass 0
Joints:
- added joint FL_calf_joint: type revolute, parent FL_thigh, child FL_calf, origin xyz=0 0 -0.213 rpy=0 0 0, axis 0 1 0, limit lower=-2.7227 upper=-0.83776 effort=35.55 velocity=20.07
- added joint FL_calflower1_joint: type fixed, parent FL_calflower, child FL_calflower1, origin xyz=-0.01 0 -0.04 rpy=0 0.48 0, axis 0 0 0
- added joint FL_calflower_joint: type fixed, parent FL_calf, child FL_calflower, origin xyz=0.020 0 -0.148 rpy=0 0.05 0, axis 0 0 0
- added joint FL_foot_joint: type fixed, parent FL_calf, child FL_foot, origin xyz=0 0 -0.213 rpy=0 0 0, axis 0 0 0
- added joint FL_hip_joint: type revolute, parent base, child FL_hip, origin xyz=0.1934 0.0465 0 rpy=0 0 0, axis 1 0 0, limit lower=-1.0472 upper=1.0472 effort=23.7 velocity=30.1
- added joint FL_thigh_joint: type revolute, parent FL_hip, child FL_thigh, origin xyz=0 0.0955 0 rpy=0 0 0, axis 0 1 0, limit lower=-1.5708 upper=3.4907 effort=23.7 velocity=30.1
- added joint FR_calf_joint: type revolute, parent FR_thigh, child FR_calf, origin xyz=0 0 -0.213 rpy=0 0 0, axis 0 1 0, limit lower=-2.7227 upper=-0.83776 effort=35.55 velocity=20.07
- added joint FR_calflower1_joint: type fixed, parent FR_calflower, child FR_calflower1, origin xyz=-0.01 0 -0.04 rpy=0 0.48 0, axis 0 0 0
- added joint FR_calflower_joint: type fixed, parent FR_calf, child FR_calflower, origin xyz=0.020 0 -0.148 rpy=0 0.05 0, axis 0 0 0
- added joint FR_foot_joint: type fixed, parent FR_calf, child FR_foot, origin xyz=0 0 -0.213 rpy=0 0 0, axis 0 0 0
- added joint FR_hip_joint: type revolute, parent base, child FR_hip, origin xyz=0.1934 -0.0465 0 rpy=0 0 0, axis 1 0 0, limit lower=-1.0472 upper=1.0472 effort=23.7 velocity=30.1
- added joint FR_thigh_joint: type revolute, parent FR_hip, child FR_thigh, origin xyz=0 -0.0955 0 rpy=0 0 0, axis 0 1 0, limit lower=-1.5708 upper=3.4907 effort=23.7 velocity=30.1
- added joint Head_lower_joint: type fixed, parent Head_upper, child Head_lower, origin xyz=0.008 0 -0.07 rpy=0 0 0, axis 0 0 0
- added joint Head_upper_joint: type fixed, parent base, child Head_upper, origin xyz=0.285 0 0.01 rpy=0 0 0, axis 0 0 0
- added joint RL_calf_joint: type revolute, parent RL_thigh, child RL_calf, origin xyz=0 0 -0.213 rpy=0 0 0, axis 0 1 0, limit lower=-2.7227 upper=-0.83776 effort=35.55 velocity=20.07
- added joint RL_calflower1_joint: type fixed, parent RL_calflower, child RL_calflower1, origin xyz=-0.01 0 -0.04 rpy=0 0.48 0, axis 0 0 0
- added joint RL_calflower_joint: type fixed, parent RL_calf, child RL_calflower, origin xyz=0.020 0 -0.148 rpy=0 0.05 0, axis 0 0 0
- added joint RL_foot_joint: type fixed, parent RL_calf, child RL_foot, origin xyz=0 0 -0.213 rpy=0 0 0, axis 0 0 0
- added joint RL_hip_joint: type revolute, parent base, child RL_hip, origin xyz=-0.1934 0.0465 0 rpy=0 0 0, axis 1 0 0, limit lower=-1.0472 upper=1.0472 effort=23.7 velocity=30.1
- added joint RL_thigh_joint: type revolute, parent RL_hip, child RL_thigh, origin xyz=0 0.0955 0 rpy=0 0 0, axis 0 1 0, limit lower=-0.5236 upper=4.5379 effort=23.7 velocity=30.1
- added joint RR_calf_joint: type revolute, parent RR_thigh, child RR_calf, origin xyz=0 0 -0.213 rpy=0 0 0, axis 0 1 0, limit lower=-2.7227 upper=-0.83776 effort=35.55 velocity=20.07
- added joint RR_calflower1_joint: type fixed, parent RR_calflower, child RR_calflower1, origin xyz=-0.01 0 -0.04 rpy=0 0.48 0, axis 0 0 0
- added joint RR_calflower_joint: type fixed, parent RR_calf, child RR_calflower, origin xyz=0.020 0 -0.148 rpy=0 0.05 0, axis 0 0 0
- added joint RR_foot_joint: type fixed, parent RR_calf, child RR_foot, origin xyz=0 0 -0.213 rpy=0 0 0, axis 0 0 0
- added joint RR_hip_joint: type revolute, parent base, child RR_hip, origin xyz=-0.1934 -0.0465 0 rpy=0 0 0, axis 1 0 0, limit lower=-1.0472 upper=1.0472 effort=23.7 velocity=30.1
- added joint RR_thigh_joint: type revolute, parent RR_hip, child RR_thigh, origin xyz=0 -0.0955 0 rpy=0 0 0, axis 0 1 0, limit lower=-0.5236 upper=4.5379 effort=23.7 velocity=30.1
- added joint imu_joint: type fixed, parent base, child imu, origin xyz=-0.02557 0 0.04232 rpy=0 0 0, axis 0 0 0
- added joint j_go2_base_arm_plate: type fixed, parent base, child plate, origin xyz=0.35 0 0.08 rpy=0 0 0
- added joint radar_joint: type fixed, parent base, child radar, origin xyz=0.28945 0 -0.046825 rpy=0 2.8782 0, axis 0 0 0

Commit message: Update Jetson GO2 runtime configuration

File: craft/robot.urdf (robot description, URDF)
Before this commit: robot go2_arm, 45 links, 44 joints
Joints:
- joint j_go2_base_arm_plate: origin xyz=0.35 0 0.08 rpy=0 0 0 -> xyz=0.32 0 0.07 rpy=0 0 0

Commit message: update

File: craft/robot.urdf (robot description, URDF)
Before this commit: robot go2_arm, 45 links, 44 joints
Joints:
- joint j_go2_base_arm_plate: origin xyz=0.32 0 0.07 rpy=0 0 0 -> xyz=0.35 0 0.08 rpy=0 0 0

Commit message: Add disturbance-aware gaze stabilization experiment framework

File: craft/robot.urdf (robot description, URDF)
Before this commit: robot go2_arm, 45 links, 44 joints
Joints:
- joint j_go2_base_arm_plate: origin xyz=0.35 0 0.08 rpy=0 0 0 -> xyz=0.1 0 0.07 rpy=0 0 0

Commit message: 1254

File: craft/robot.urdf (robot description, URDF)
Before this commit: robot go2_arm, 45 links, 44 joints
Joints:
- joint j_housing_wedge: origin xyz=0 0 0.128 rpy=0 0 0 -> xyz=0 0 0.155 rpy=0 0 0

Commit message: choi jeok hwa

File: craft/robot.urdf (robot description, URDF)
Before this commit: robot go2_arm, 45 links, 44 joints
Links:
- added link camera, mass 0.05; visual mesh filename=../assets/camera/camera_mesh.obj
Joints:
- added joint j_gripper_base_camera: type fixed, parent gripper_base, child camera, origin xyz=-0.025 0 -0.00495 rpy=-3.14159265 0 -1.57079633, axis 0 -1 0
- joint j_gripper_base_claw_left: origin xyz=0 0 0 rpy=1.57079633 0 0 -> xyz=0.01046 -0.02587 -0.019 rpy=1.57079633 0 0
- joint j_gripper_base_claw_right: origin xyz=0 0 0 rpy=1.57079633 0 0 -> xyz=0.01046 0.02587 -0.019 rpy=1.57079633 0 0

Commit message: UI so dirty!

File: craft/robot.urdf (robot description, URDF)
Before this commit: robot go2_arm, 46 links, 45 joints
Links:
- added link camera_optical_marker, mass 0.001; visual mesh filename=../assets/camera_optical_marker/camera_optical_marker_mesh.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
Joints:
- added joint j_camera_optical_marker: type fixed, parent camera, child camera_optical_marker, origin xyz=-0.037 0 0.02505 rpy=0 0 0, axis 1 0 0

Commit message: 2026-06-27 06:00

File: craft/robot.urdf (robot description, URDF)
Before this commit: robot go2_arm, 47 links, 46 joints
Links:
- removed link camera_optical_marker
Joints:
- removed joint j_camera_optical_marker
