Commit message: 2026-06-28 17:51

File: crafts/arm.urdf (robot description, URDF)
Before this commit: robot Robot, 17 links, 16 joints
Joints:
- joint j_plate_housing: limit lower=-0.23 upper=0.01 effort=200 velocity=3 -> lower=-0.23 upper=0 effort=200 velocity=3

File: crafts/robot.urdf (robot description, URDF)
Before this commit: robot go2_arm, 46 links, 45 joints
Joints:
- joint j_plate_housing: limit lower=-0.23 upper=0.01 effort=200 velocity=3 -> lower=-0.23 upper=0 effort=200 velocity=3
