Commit message: update

File: crafts/arm.urdf (robot description, URDF)
Before this commit: robot Robot, 17 links, 16 joints
Links:
- link camera: mass 0.05 -> 0.005
- link gripper_base: mass 0.15 -> 0.015
- link gripper_claw_left: mass 0.05 -> 0.005
- link gripper_claw_right: mass 0.05 -> 0.005
- link housing: mass 1.8 -> 0.18
- link node0: mass 0.15 -> 0.015
- link node1: mass 0.15 -> 0.015
- link node2: mass 0.15 -> 0.015
- link node3: mass 0.15 -> 0.015
- link node4: mass 0.15 -> 0.015
- link node5: mass 0.15 -> 0.015
- link node6: mass 0.15 -> 0.015
- link node7: mass 0.15 -> 0.015
- link node8: mass 0.15 -> 0.015
- link node9: mass 0.15 -> 0.015
- link plate: mass 1.5 -> 0.15
- link wedge: mass 0.1 -> 0.01

File: crafts/go2_colored.urdf (robot description, URDF)
Before this commit: robot go2_description, 29 links, 28 joints
Links:
- link FL_calf: geometry collision cylinder length=0.12 radius=0.012; visual mesh filename=/Users/hwancheolkang/Workspace/elesim/assets/go2/dae/calf.d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
- link FL_foot: geometry collision sphere radius=0.022; visual mesh filename=/Users/hwancheolkang/Workspace/elesim/assets/go2/dae/foot.d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
- link FL_hip: geometry collision cylinder length=0.04 radius=0.046; visual mesh filename=/Users/hwancheolkang/Workspace/elesim/assets/go2/dae/hip.dae
- link FL_thigh: geometry collision box size=0.11 0.0245 0.034; visual mesh filename=/Users/hwancheolkang/Workspace/elesim/assets/go2/dae/thigh.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
- link FR_calf: geometry collision cylinder length=0.12 radius=0.013; visual mesh filename=/Users/hwancheolkang/Workspace/elesim/assets/go2/dae/calf_m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
- link FR_foot: geometry collision sphere radius=0.022; visual mesh filename=/Users/hwancheolkang/Workspace/elesim/assets/go2/dae/foot.d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
- link FR_hip: geometry collision cylinder length=0.04 radius=0.046; visual mesh filename=/Users/hwancheolkang/Workspace/elesim/assets/go2/dae/hip.dae
- link FR_thigh: geometry collision box size=0.11 0.0245 0.034; visual mesh filename=/Users/hwancheolkang/Workspace/elesim/assets/go2/dae/thigh_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
- link RL_calf: geometry collision cylinder length=0.12 radius=0.013; visual mesh filename=/Users/hwancheolkang/Workspace/elesim/assets/go2/dae/calf.d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
- link RL_foot: geometry collision sphere radius=0.022; visual mesh filename=/Users/hwancheolkang/Workspace/elesim/assets/go2/dae/foot.d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
- link RL_hip: geometry collision cylinder length=0.04 radius=0.046; visual mesh filename=/Users/hwancheolkang/Workspace/elesim/assets/go2/dae/hip.dae
- link RL_thigh: geometry collision box size=0.11 0.0245 0.034; visual mesh filename=/Users/hwancheolkang/Workspace/elesim/assets/go2/dae/thigh.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
- link RR_calf: geometry collision cylinder length=0.12 radius=0.013; visual mesh filename=/Users/hwancheolkang/Workspace/elesim/assets/go2/dae/calf_m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
- link RR_foot: geometry collision sphere radius=0.022; visual mesh filename=/Users/hwancheolkang/Workspace/elesim/assets/go2/dae/foot.d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
- link RR_hip: geometry collision cylinder length=0.04 radius=0.046; visual mesh filename=/Users/hwancheolkang/Workspace/elesim/assets/go2/dae/hip.dae
- link RR_thigh: geometry collision box size=0.11 0.0245 0.034; visual mesh filename=/Users/hwancheolkang/Workspace/elesim/assets/go2/dae/thigh_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
- link base: geometry collision box size=0.3762 0.0935 0.114; visual mesh filename=/Users/hwancheolkang/Workspace/elesim/assets/go2/dae/base.d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

File: crafts/robot.urdf (robot description, URDF)
Before this commit: robot go2_arm, 46 links, 45 joints
Links:
- link FL_calf: geometry collision cylinder length=0.12 radius=0.012; visual mesh filename=/Users/hwancheolkang/Workspace/elesim/assets/go2/dae/calf.d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
- link FL_foot: geometry collision sphere radius=0.022; visual mesh filename=/Users/hwancheolkang/Workspace/elesim/assets/go2/dae/foot.d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
- link FL_hip: geometry collision cylinder length=0.04 radius=0.046; visual mesh filename=/Users/hwancheolkang/Workspace/elesim/assets/go2/dae/hip.dae
- link FL_thigh: geometry collision box size=0.11 0.0245 0.034; visual mesh filename=/Users/hwancheolkang/Workspace/elesim/assets/go2/dae/thigh.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
- link FR_calf: geometry collision cylinder length=0.12 radius=0.013; visual mesh filename=/Users/hwancheolkang/Workspace/elesim/assets/go2/dae/calf_m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
- link FR_foot: geometry collision sphere radius=0.022; visual mesh filename=/Users/hwancheolkang/Workspace/elesim/assets/go2/dae/foot.d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
- link FR_hip: geometry collision cylinder length=0.04 radius=0.046; visual mesh filename=/Users/hwancheolkang/Workspace/elesim/assets/go2/dae/hip.dae
- link FR_thigh: geometry collision box size=0.11 0.0245 0.034; visual mesh filename=/Users/hwancheolkang/Workspace/elesim/assets/go2/dae/thigh_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
- link RL_calf: geometry collision cylinder length=0.12 radius=0.013; visual mesh filename=/Users/hwancheolkang/Workspace/elesim/assets/go2/dae/calf.d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
- link RL_foot: geometry collision sphere radius=0.022; visual mesh filename=/Users/hwancheolkang/Workspace/elesim/assets/go2/dae/foot.d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
- link RL_hip: geometry collision cylinder length=0.04 radius=0.046; visual mesh filename=/Users/hwancheolkang/Workspace/elesim/assets/go2/dae/hip.dae
- link RL_thigh: geometry collision box size=0.11 0.0245 0.034; visual mesh filename=/Users/hwancheolkang/Workspace/elesim/assets/go2/dae/thigh.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
- link RR_calf: geometry collision cylinder length=0.12 radius=0.013; visual mesh filename=/Users/hwancheolkang/Workspace/elesim/assets/go2/dae/calf_m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
- link RR_foot: geometry collision sphere radius=0.022; visual mesh filename=/Users/hwancheolkang/Workspace/elesim/assets/go2/dae/foot.d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
- link RR_hip: geometry collision cylinder length=0.04 radius=0.046; visual mesh filename=/Users/hwancheolkang/Workspace/elesim/assets/go2/dae/hip.dae
- link RR_thigh: geometry collision box size=0.11 0.0245 0.034; visual mesh filename=/Users/hwancheolkang/Workspace/elesim/assets/go2/dae/thigh_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
- link base: geometry collision box size=0.3762 0.0935 0.114; visual mesh filename=/Users/hwancheolkang/Workspace/elesim/assets/go2/dae/base.d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
- link camera: mass 0.05 -> 0.005
Joints:
- joint j_go2_base_arm_plate: origin xyz=0.315 0 0.08 rpy=0 0 0 -> xyz=0.1 0 0.07 rpy=0 0 0
