Commit message: Restore Pitch Preview on behaviors/gaze layout after origin/main merge.
Port preview MPC-lite, pitch/gait preview gaze modes, experiment tooling, and walking metrics logging to the refactored engine paths.

File: crafts/robot.urdf (robot description, URDF)
Before this commit: robot go2_arm, 46 links, 45 joints
Links:
- link gripper_base: mass 0.15 -> 0.015
- link gripper_claw_left: mass 0.05 -> 0.005
- link gripper_claw_right: mass 0.05 -> 0.005
- link housing: mass 1.8 -> 0.18
- link node0: mass 0.15 -> 0.015
- link node1: mass 0.15 -> 0.015
- link node2: mass 0.15 -> 0.015
- link node3: mass 0.15 -> 0.015
- link node4: mass 0.15 -> 0.015
- link node5: mass 0.15 -> 0.015
- link node6: mass 0.15 -> 0.015
- link node7: mass 0.15 -> 0.015
- link node8: mass 0.15 -> 0.015
- link node9: mass 0.15 -> 0.015
- link plate: mass 1.5 -> 0.15
- link wedge: mass 0.1 -> 0.01
Joints:
- joint j_go2_base_arm_plate: origin xyz=0.1 0 0.07 rpy=0 0 0 -> xyz=0.315 0 0.08 rpy=0 0 0

Commit message: update

File: crafts/robot.urdf (robot description, URDF)
Before this commit: robot go2_arm, 46 links, 45 joints
Joints:
- joint j_go2_base_arm_plate: origin xyz=0.1 0 0.07 rpy=0 0 0 -> xyz=0.35 0 0.08 rpy=0 0 0
