Commit message: big change

File: model/bundles/default/arm.urdf (robot description, URDF)
Before this commit: robot Robot, 17 links, 16 joints
Links:
- link camera: geometry visual mesh filename=assets/camera/camera_mesh.obj
- link gripper_base: geometry collision mesh filename=assets/gripper_base/gripper_base_mesh.obj; visual mesh filename=assets/gripper_base/gripper_base_mesh.obj
- link gripper_claw_left: geometry collision mesh filename=assets/gripper_claw_left/gripper_claw_left_mesh.obj; visual mesh filename=assets/gripper_claw_left/gripper_claw_left_mesh.obj
- link gripper_claw_right: geometry collision mesh filename=assets/gripper_claw_right/gripper_claw_right_mesh.obj; visual mesh filename=assets/gripper_claw_right/gripper_claw_right_mesh.obj
- link housing: geometry collision mesh filename=assets/housing/housing_mesh.obj; visual mesh filename=assets/housing/housing_mesh.obj
- link node0: geometry collision mesh filename=assets/node/node_mesh.obj; visual mesh filename=assets/node/node_mesh.obj
- link node1: geometry collision mesh filename=assets/node/node_mesh.obj; visual mesh filename=assets/node/node_mesh.obj
- link node2: geometry collision mesh filename=assets/node/node_mesh.obj; visual mesh filename=assets/node/node_mesh.obj
- link node3: geometry collision mesh filename=assets/node/node_mesh.obj; visual mesh filename=assets/node/node_mesh.obj
- link node4: geometry collision mesh filename=assets/node/node_mesh.obj; visual mesh filename=assets/node/node_mesh.obj
- link node5: geometry collision mesh filename=assets/node/node_mesh.obj; visual mesh filename=assets/node/node_mesh.obj
- link node6: geometry collision mesh filename=assets/node/node_mesh.obj; visual mesh filename=assets/node/node_mesh.obj
- link node7: geometry collision mesh filename=assets/node/node_mesh.obj; visual mesh filename=assets/node/node_mesh.obj
- link node8: geometry collision mesh filename=assets/node/node_mesh.obj; visual mesh filename=assets/node/node_mesh.obj
- link node9: geometry collision mesh filename=assets/node_end/node_end_mesh.obj; visual mesh filename=assets/node_end/node_end_mesh.obj
- link plate: geometry collision mesh filename=assets/plate/plate_mesh.obj; visual mesh filename=assets/plate/plate_mesh.obj
- link wedge: geometry collision mesh filename=assets/wedge/wedge_mesh.obj; visual mesh filename=assets/wedge/wedge_mesh.obj

File: model/bundles/default/robot.urdf (robot description, URDF)
Before this commit: robot go2_arm, 46 links, 45 joints
Links:
- link FL_calf: geometry collision cylinder length=0.12 radius=0.012; visual mesh filename=assets/go2/dae/calf.dae
- link FL_foot: geometry collision sphere radius=0.022; visual mesh filename=assets/go2/dae/foot.dae
- link FL_hip: geometry collision cylinder length=0.04 radius=0.046; visual mesh filename=assets/go2/dae/hip.dae
- link FL_thigh: geometry collision box size=0.11 0.0245 0.034; visual mesh filename=assets/go2/dae/thigh.dae
- link FR_calf: geometry collision cylinder length=0.12 radius=0.013; visual mesh filename=assets/go2/dae/calf_mirror.dae
- link FR_foot: geometry collision sphere radius=0.022; visual mesh filename=assets/go2/dae/foot.dae
- link FR_hip: geometry collision cylinder length=0.04 radius=0.046; visual mesh filename=assets/go2/dae/hip.dae
- link FR_thigh: geometry collision box size=0.11 0.0245 0.034; visual mesh filename=assets/go2/dae/thigh_mirror.dae
- link RL_calf: geometry collision cylinder length=0.12 radius=0.013; visual mesh filename=assets/go2/dae/calf.dae
- link RL_foot: geometry collision sphere radius=0.022; visual mesh filename=assets/go2/dae/foot.dae
- link RL_hip: geometry collision cylinder length=0.04 radius=0.046; visual mesh filename=assets/go2/dae/hip.dae
- link RL_thigh: geometry collision box size=0.11 0.0245 0.034; visual mesh filename=assets/go2/dae/thigh.dae
- link RR_calf: geometry collision cylinder length=0.12 radius=0.013; visual mesh filename=assets/go2/dae/calf_mirror.dae
- link RR_foot: geometry collision sphere radius=0.022; visual mesh filename=assets/go2/dae/foot.dae
- link RR_hip: geometry collision cylinder length=0.04 radius=0.046; visual mesh filename=assets/go2/dae/hip.dae
- link RR_thigh: geometry collision box size=0.11 0.0245 0.034; visual mesh filename=assets/go2/dae/thigh_mirror.dae
- link base: geometry collision box size=0.3762 0.0935 0.114; visual mesh filename=assets/go2/dae/base.dae
- link camera: geometry visual mesh filename=assets/camera/camera_mesh.obj
- link gripper_base: geometry collision mesh filename=assets/gripper_base/gripper_base_mesh.obj; visual mesh filename=assets/gripper_base/gripper_base_mesh.obj
- link gripper_claw_left: geometry collision mesh filename=assets/gripper_claw_left/gripper_claw_left_mesh.obj; visual mesh filename=assets/gripper_claw_left/gripper_claw_left_mesh.obj
- link gripper_claw_right: geometry collision mesh filename=assets/gripper_claw_right/gripper_claw_right_mesh.obj; visual mesh filename=assets/gripper_claw_right/gripper_claw_right_mesh.obj
- link housing: geometry collision mesh filename=assets/housing/housing_mesh.obj; visual mesh filename=assets/housing/housing_mesh.obj
- link node0: geometry collision mesh filename=assets/node/node_mesh.obj; visual mesh filename=assets/node/node_mesh.obj
- link node1: geometry collision mesh filename=assets/node/node_mesh.obj; visual mesh filename=assets/node/node_mesh.obj
- link node2: geometry collision mesh filename=assets/node/node_mesh.obj; visual mesh filename=assets/node/node_mesh.obj
- link node3: geometry collision mesh filename=assets/node/node_mesh.obj; visual mesh filename=assets/node/node_mesh.obj
- link node4: geometry collision mesh filename=assets/node/node_mesh.obj; visual mesh filename=assets/node/node_mesh.obj
- link node5: geometry collision mesh filename=assets/node/node_mesh.obj; visual mesh filename=assets/node/node_mesh.obj
- link node6: geometry collision mesh filename=assets/node/node_mesh.obj; visual mesh filename=assets/node/node_mesh.obj
- link node7: geometry collision mesh filename=assets/node/node_mesh.obj; visual mesh filename=assets/node/node_mesh.obj
- link node8: geometry collision mesh filename=assets/node/node_mesh.obj; visual mesh filename=assets/node/node_mesh.obj
- link node9: geometry collision mesh filename=assets/node_end/node_end_mesh.obj; visual mesh filename=assets/node_end/node_end_mesh.obj
- link plate: geometry collision mesh filename=assets/plate/plate_mesh.obj; visual mesh filename=assets/plate/plate_mesh.obj
- link wedge: geometry collision mesh filename=assets/wedge/wedge_mesh.obj; visual mesh filename=assets/wedge/wedge_mesh.obj
Joints:
- joint j_go2_base_arm_plate: origin xyz=0.1 0 0.07 rpy=0 0 0 -> xyz=0.35 0 0.08 rpy=0 0 0

Commit message: Add ZED Mini camera profile with D435 fallback

File: model/bundles/default/arm.urdf (robot description, URDF)
Before this commit: robot Robot, 17 links, 16 joints
Links:
- link camera: mass 0.005 -> 0.0629
Joints:
- joint j_gripper_base_camera: axis 0 -1 0 -> 0 0 -1; origin xyz=-0.025 0 -0.00495 rpy=-3.14159265 0 -1.57079633 -> xyz=-0.042062 -0.00632 -0.005021 rpy=-1.57079633 -2.22044605e-16 1.57079633

File: model/bundles/default/robot.urdf (robot description, URDF)
Before this commit: robot go2_arm, 46 links, 45 joints
Links:
- link camera: mass 0.005 -> 0.0629
Joints:
- joint j_gripper_base_camera: axis 0 -1 0 -> 0 0 -1; origin xyz=-0.025 0 -0.00495 rpy=-3.14159265 0 -1.57079633 -> xyz=-0.042062 -0.00632 -0.005021 rpy=-1.57079633 -2.22044605e-16 1.57079633
