Commit message: Fix linear calibration and GO2 plate alignment; simplify setup wizard

File: payload/data/models/assemblies/d435/arm.urdf (robot description, URDF)
Before this commit: robot Robot, 17 links, 16 joints
Joints:
- joint j_plate_housing: limit lower=-0.23 upper=0 effort=200 velocity=3 -> lower=-0.166666667 upper=0 effort=200 velocity=3

File: payload/data/models/assemblies/d435/robot.urdf (robot description, URDF)
Before this commit: robot go2_arm, 46 links, 45 joints
Joints:
- joint j_go2_base_arm_plate: origin xyz=0.35 0 0.08 rpy=0 0 0 -> xyz=0.315 0 0.087 rpy=0 0 0
- joint j_plate_housing: limit lower=-0.23 upper=0 effort=200 velocity=3 -> lower=-0.166666667 upper=0 effort=200 velocity=3

File: payload/data/models/assemblies/zed-mini/arm.urdf (robot description, URDF)
Before this commit: robot Robot, 17 links, 16 joints
Joints:
- joint j_plate_housing: limit lower=-0.23 upper=0 effort=200 velocity=3 -> lower=-0.166666667 upper=0 effort=200 velocity=3

File: payload/data/models/assemblies/zed-mini/robot.urdf (robot description, URDF)
Before this commit: robot go2_arm, 46 links, 45 joints
Joints:
- joint j_go2_base_arm_plate: origin xyz=0.35 0 0.08 rpy=0 0 0 -> xyz=0.315 0 0.087 rpy=0 0 0
- joint j_plate_housing: limit lower=-0.23 upper=0 effort=200 velocity=3 -> lower=-0.166666667 upper=0 effort=200 velocity=3

Commit message: Share calibrated linear operating limits across runtime and training

File: payload/data/models/assemblies/d435/arm.urdf (robot description, URDF)
Before this commit: robot Robot, 17 links, 16 joints
Joints:
- joint j_plate_housing: limit lower=-0.166666667 upper=0 effort=200 velocity=3 -> lower=-0.142 upper=0 effort=200 velocity=3

File: payload/data/models/assemblies/d435/robot.urdf (robot description, URDF)
Before this commit: robot go2_arm, 46 links, 45 joints
Joints:
- joint j_plate_housing: limit lower=-0.166666667 upper=0 effort=200 velocity=3 -> lower=-0.142 upper=0 effort=200 velocity=3

File: payload/data/models/assemblies/zed-mini/arm.urdf (robot description, URDF)
Before this commit: robot Robot, 17 links, 16 joints
Joints:
- joint j_plate_housing: limit lower=-0.166666667 upper=0 effort=200 velocity=3 -> lower=-0.142 upper=0 effort=200 velocity=3

File: payload/data/models/assemblies/zed-mini/robot.urdf (robot description, URDF)
Before this commit: robot go2_arm, 46 links, 45 joints
Joints:
- joint j_plate_housing: limit lower=-0.166666667 upper=0 effort=200 velocity=3 -> lower=-0.142 upper=0 effort=200 velocity=3

Commit message: Add arm trajectory planning and contact hold

File: payload/data/models/assemblies/d435/arm.urdf (robot description, URDF)
Before this commit: robot Robot, 17 links, 16 joints
Joints:
- joint j_plate_housing: limit lower=-0.142 upper=0 effort=200 velocity=3 -> lower=-0.172666667 upper=0 effort=200 velocity=3

File: payload/data/models/assemblies/d435/robot.urdf (robot description, URDF)
Before this commit: robot go2_arm, 46 links, 45 joints
Joints:
- joint j_plate_housing: limit lower=-0.142 upper=0 effort=200 velocity=3 -> lower=-0.172666667 upper=0 effort=200 velocity=3

File: payload/data/models/assemblies/zed-mini/arm.urdf (robot description, URDF)
Before this commit: robot Robot, 17 links, 16 joints
Joints:
- joint j_plate_housing: limit lower=-0.142 upper=0 effort=200 velocity=3 -> lower=-0.172666667 upper=0 effort=200 velocity=3

File: payload/data/models/assemblies/zed-mini/robot.urdf (robot description, URDF)
Before this commit: robot go2_arm, 46 links, 45 joints
Joints:
- joint j_plate_housing: limit lower=-0.142 upper=0 effort=200 velocity=3 -> lower=-0.172666667 upper=0 effort=200 velocity=3

File: payload/data/models/planning/zed-mini/arm.urdf (robot description, URDF)
Before this commit: robot Robot, 18 links, 17 joints
Joints:
- joint j_housing_wedge: limit lower=-1.5707963267948966 upper=1.5707963267948966 effort=200 velocity=0.35 -> lower=-1.5707963267948966 upper=1.5707963267948966 effort=200 velocity=3.5
- joint j_node0_node1: limit lower=-0.6283185307179586 upper=0.6283185307179586 effort=200 velocity=0.1 -> lower=-0.6283185307179586 upper=0.6283185307179586 effort=200 velocity=1.0
- joint j_node1_node2: limit lower=-0.6283185307179586 upper=0.6283185307179586 effort=200 velocity=0.1 -> lower=-0.6283185307179586 upper=0.6283185307179586 effort=200 velocity=1.0
- joint j_node2_node3: limit lower=-0.6283185307179586 upper=0.6283185307179586 effort=200 velocity=0.1 -> lower=-0.6283185307179586 upper=0.6283185307179586 effort=200 velocity=1.0
- joint j_node3_node4: limit lower=-0.6283185307179586 upper=0.6283185307179586 effort=200 velocity=0.1 -> lower=-0.6283185307179586 upper=0.6283185307179586 effort=200 velocity=1.0
- joint j_node4_node5: limit lower=-0.6283185307179586 upper=0.6283185307179586 effort=200 velocity=0.1 -> lower=-0.6283185307179586 upper=0.6283185307179586 effort=200 velocity=1.0
- joint j_node5_node6: limit lower=-0.6283185307179586 upper=0.6283185307179586 effort=200 velocity=0.1 -> lower=-0.6283185307179586 upper=0.6283185307179586 effort=200 velocity=1.0
- joint j_node6_node7: limit lower=-0.6283185307179586 upper=0.6283185307179586 effort=200 velocity=0.1 -> lower=-0.6283185307179586 upper=0.6283185307179586 effort=200 velocity=1.0
- joint j_node7_node8: limit lower=-0.6283185307179586 upper=0.6283185307179586 effort=200 velocity=0.1 -> lower=-0.6283185307179586 upper=0.6283185307179586 effort=200 velocity=1.0
- joint j_node8_node9: limit lower=-0.6283185307179586 upper=0.6283185307179586 effort=200 velocity=0.1 -> lower=-0.6283185307179586 upper=0.6283185307179586 effort=200 velocity=1.0
- joint j_plate_housing: limit lower=-0.142 upper=0.0 effort=200 velocity=0.02 -> lower=-0.17266666666666666 upper=0.0 effort=200 velocity=0.2
- joint j_wedge_node0: limit lower=-0.6283185307179586 upper=0.6283185307179586 effort=200 velocity=0.1 -> lower=-0.6283185307179586 upper=0.6283185307179586 effort=200 velocity=1.0

Commit message: Align 4DOF linear range with oct27 policy

File: payload/data/models/assemblies/d435/arm.urdf (robot description, URDF)
Before this commit: robot Robot, 17 links, 16 joints
Joints:
- joint j_plate_housing: limit lower=-0.172666667 upper=0 effort=200 velocity=3 -> lower=-0.23 upper=0 effort=200 velocity=3

File: payload/data/models/assemblies/d435/robot.urdf (robot description, URDF)
Before this commit: robot go2_arm, 46 links, 45 joints
Joints:
- joint j_plate_housing: limit lower=-0.172666667 upper=0 effort=200 velocity=3 -> lower=-0.23 upper=0 effort=200 velocity=3

File: payload/data/models/assemblies/zed-mini/arm.urdf (robot description, URDF)
Before this commit: robot Robot, 17 links, 16 joints
Joints:
- joint j_plate_housing: limit lower=-0.172666667 upper=0 effort=200 velocity=3 -> lower=-0.23 upper=0 effort=200 velocity=3

File: payload/data/models/assemblies/zed-mini/robot.urdf (robot description, URDF)
Before this commit: robot go2_arm, 46 links, 45 joints
Joints:
- joint j_plate_housing: limit lower=-0.172666667 upper=0 effort=200 velocity=3 -> lower=-0.23 upper=0 effort=200 velocity=3

File: payload/data/models/planning/zed-mini/arm.urdf (robot description, URDF)
Before this commit: robot Robot, 18 links, 17 joints
Joints:
- joint j_plate_housing: limit lower=-0.17266666666666666 upper=0.0 effort=200 velocity=0.2 -> lower=-0.23 upper=0.0 effort=200 velocity=0.2

Commit message: Apply field fixes and complete Sim scanning workflow
Keep the 1.5 degrees/mm linear calibration and 260-degree cap across runtime settings and model artifacts. Preserve installed Robot calibration and host facts, restore the pinned wrap policy, and incorporate Jetson, presentation, GPU and lifecycle fixes.

Add replaceable reconstruction model slots, immutable scene artifacts, and the Sim-only active multiview scan with UI controls, fresh settled captures, silhouettes and point-cloud fusion. Fix cancellation, mirror pinning, legacy UI preflight, pending GPU drafts and reassigned role policies found during review.

Validation includes host Pilot, UI, protocol, targeted Sim and setup/release tests; the review follow-up passes 277 Python and 8 JavaScript tests. Canonical ROS/GPU/hardware and isolated release gates remain unrun as recorded in docs/status.md. Preserve plzread.md as the original field-diff reference.

File: payload/data/models/assemblies/d435/arm.urdf (robot description, URDF)
Before this commit: robot Robot, 17 links, 16 joints
Joints:
- joint j_plate_housing: limit lower=-0.23 upper=0 effort=200 velocity=3 -> lower=-0.173333333 upper=0 effort=200 velocity=3

File: payload/data/models/assemblies/d435/robot.urdf (robot description, URDF)
Before this commit: robot go2_arm, 46 links, 45 joints
Joints:
- joint j_plate_housing: limit lower=-0.23 upper=0 effort=200 velocity=3 -> lower=-0.173333333 upper=0 effort=200 velocity=3

File: payload/data/models/assemblies/zed-mini/arm.urdf (robot description, URDF)
Before this commit: robot Robot, 17 links, 16 joints
Joints:
- joint j_plate_housing: limit lower=-0.23 upper=0 effort=200 velocity=3 -> lower=-0.173333333 upper=0 effort=200 velocity=3

File: payload/data/models/assemblies/zed-mini/robot.urdf (robot description, URDF)
Before this commit: robot go2_arm, 46 links, 45 joints
Joints:
- joint j_plate_housing: limit lower=-0.23 upper=0 effort=200 velocity=3 -> lower=-0.173333333 upper=0 effort=200 velocity=3

File: payload/data/models/planning/zed-mini/arm.urdf (robot description, URDF)
Before this commit: robot Robot, 18 links, 17 joints
Joints:
- joint j_plate_housing: limit lower=-0.23 upper=0.0 effort=200 velocity=0.2 -> lower=-0.17333333333333334 upper=0.0 effort=200 velocity=0.2
